File: schematic/fumisAdapter.sch (KiCad schematic (older format))
At the start: 18 parts, among them Q1 BC847, Q2 BC847, U1 SI8621

Commit message: Update schematic
Parts:
- removed D2: D, symbol Device:D
- added D2: 0.3V, symbol Device:D_Schottky
- added J?: HalfMode, Pin_Headers:Pin_Header_Straight_1x03_Pitch2.54mm, symbol Connector_Generic:Conn_01x03
- C1, C2: footprint (none) -> Capacitors_SMD:C_0805_HandSoldering
- D1, D3: value LED -> RED LED; footprint (none) -> Resistors_SMD:R_0805_HandSoldering
- J1: renamed from J?; footprint (none) -> Connect:RJ12_E
- J2: renamed from J?; value Conn_01x04 -> MCU UART
- Q1, Q2: value BC847 -> BC847B
- R1, R2, R6, R7, R8: footprint (none) -> Resistors_SMD:R_0805_HandSoldering
- R3: value 2.8K -> 2K; footprint (none) -> Resistors_SMD:R_0805_HandSoldering
- R4: value 2.8K -> 2K
- U1: footprint (none) -> Housings_SOIC:SOIC-8_3.9x4.9mm_Pitch1.27mm
Connections:
- net labels added: Q2B, Rx, Tx-RxH
- wire segments 26 -> 81
- no-connect marks 0 -> 1
Other:
- moved on the sheet: C1, C2, D1, D3, Q1, Q2, R1, R2, R3, R4, R5, R8

Commit message: Update schematic
Parts:
- J2: footprint (none) -> Pin_Headers:Pin_Header_Angled_1x04_Pitch2.54mm
- gave numbers to parts that had none: 1
Other:
- note added: "Default Mode : no jumper\nLabtool mode : 2-3 jumper"
Changed lines of the file:
@@
 F 0 "J2" H 5980 2042 50  0000 L CNN
 F 1 "MCU UART" H 5980 1951 50  0000 L CNN
-F 2 "" H 5900 2050 50  0001 C CNN
+F 2 "Pin_Headers:Pin_Header_Angled_1x04_Pitch2.54mm" H 5900 2050 50  0001 C CNN
 F 3 "~" H 5900 2050 50  0001 C CNN
 	1    5900 2050
@@
 NoConn ~ 1450 1700
 $Comp
-L Connector_Generic:Conn_01x03 J?
+L Connector_Generic:Conn_01x03 J3
 U 1 1 5E125751
 P 1250 3450
-F 0 "J?" V 1122 3262 50  0000 R CNN
+F 0 "J3" V 1122 3262 50  0000 R CNN
 F 1 "HalfMode" V 1213 3262 50  0000 R CNN
 F 2 "Pin_Headers:Pin_Header_Straight_1x03_Pitch2.54mm" H 1250 3450 50  0001 C CNN
@@
 Wire Wire Line
 	3200 2250 3350 2250
+Text Notes 1800 3700 2    50   ~ 0
+Default Mode : no jumper\nLabtool mode : 2-3 jumper
 $EndSCHEMATC

Commit message: Update schematic
Parts:
- D2: value 0.3V -> SS34; footprint (none) -> Diodes_SMD:D_SMA
- J2: footprint Pin_Headers:Pin_Header_Angled_1x04_Pitch2.54mm -> Pin_Headers:Pin_Header_Straight_1x04_Pitch2.54mm
- Q1, Q2: footprint Package_TO_SOT_SMD:SOT-23 -> TO_SOT_Packages_SMD:SOT-23
- R4, R5: footprint (none) -> Resistors_SMD:R_0805_HandSoldering
Changed lines of the file:
@@
 F 0 "Q2" H 1991 2846 50  0000 L CNN
 F 1 "BC847B" H 1991 2755 50  0000 L CNN
-F 2 "Package_TO_SOT_SMD:SOT-23" H 2000 2725 50  0001 L CIN
+F 2 "TO_SOT_Packages_SMD:SOT-23" H 2000 2725 50  0001 L CIN
 F 3 "http://www.infineon.com/dgdl/Infineon-BC847SERIES_BC848SERIES_BC849SERIES_BC850SERIES-DS-v01_01-en.pdf?fileId=db3a304314dca389011541d4630a1657" H 1800 2800 50  0001 L CNN
 	1    1800 2800
@@
 F 0 "J2" H 5980 2042 50  0000 L CNN
 F 1 "MCU UART" H 5980 1951 50  0000 L CNN
-F 2 "Pin_Headers:Pin_Header_Angled_1x04_Pitch2.54mm" H 5900 2050 50  0001 C CNN
+F 2 "Pin_Headers:Pin_Header_Straight_1x04_Pitch2.54mm" H 5900 2050 50  0001 C CNN
 F 3 "~" H 5900 2050 50  0001 C CNN
 	1    5900 2050
@@
 P 2500 2250
 F 0 "D2" H 2500 2350 50  0000 C CNN
-F 1 "0.3V" H 2500 2450 50  0000 C CNN
-F 2 "" H 2500 2250 50  0001 C CNN
+F 1 "SS34" H 2500 2450 50  0000 C CNN
+F 2 "Diodes_SMD:D_SMA" H 2500 2250 50  0001 C CNN
 F 3 "~" H 2500 2250 50  0001 C CNN
 	1    2500 2250
@@
 F 0 "R5" V 2950 3050 50  0000 C CNN
 F 1 "2K" V 2850 3050 50  0000 C CNN
-F 2 "" V 2780 3050 50  0001 C CNN
+F 2 "Resistors_SMD:R_0805_HandSoldering" V 2780 3050 50  0001 C CNN
 F 3 "~" H 2850 3050 50  0001 C CNN
 	1    2850 3050
@@
 F 0 "R4" V 3100 3300 50  0000 C CNN
 F 1 "2K" V 3200 3300 50  0000 C CNN
-F 2 "" V 3130 3300 50  0001 C CNN
+F 2 "Resistors_SMD:R_0805_HandSoldering" V 3130 3300 50  0001 C CNN
 F 3 "~" H 3200 3300 50  0001 C CNN
 	1    3200 3300
@@
 F 0 "Q1" H 3141 3546 50  0000 L CNN
 F 1 "BC847B" H 3141 3455 50  0000 L CNN
-F 2 "Package_TO_SOT_SMD:SOT-23" H 3150 3425 50  0001 L CIN
+F 2 "TO_SOT_Packages_SMD:SOT-23" H 3150 3425 50  0001 L CIN
 F 3 "http://www.infineon.com/dgdl/Infineon-BC847SERIES_BC848SERIES_BC849SERIES_BC850SERIES-DS-v01_01-en.pdf?fileId=db3a304314dca389011541d4630a1657" H 2950 3500 50  0001 L CNN
 	1    2950 3500
